File: Main.sch (KiCad schematic (older format))
At the start: 27 parts, among them U2 STM32F407VGTx, Y2 8MHz

Commit message: Use smd oscilator Add testpoints Use different power networks
Parts:
- L1: footprint Resistors_SMD:R_0603 -> MF_Passives:MF_Passives-L1210; MFR TDK -> Taiyo Yuden; SPN 810-MLZ1608N100L -> MF-IND-1210-10uH; SPR Mouser -> Macrofab
- Y2: footprint Crystals:Crystal_HC49-U_Vertical -> Crystals:Crystal_SMD_ABM3B; MFR Fox -> Abracon; MPN FOXSLF/080-20 -> ABM3B-8.000MHZ-10-1UT; SPN 559-FOXS080-20-LF -> 815-ABM3B-8.0-10-1UT
Changed lines of the file:
@@
 LIBS:valves
 LIBS:stm32
+LIBS:MF_Passives
 LIBS:tmb_musicplayer-cache
 EELAYER 25 0
@@
 F 0 "Y2" H 1750 2900 50  0000 C CNN
 F 1 "8MHz" V 1750 2750 50  0000 C CNN
-F 2 "Crystals:Crystal_HC49-U_Vertical" H 1750 2750 50  0001 C CNN
+F 2 "Crystals:Crystal_SMD_ABM3B" H 1750 2750 50  0001 C CNN
 F 3 "http://www.mouser.com/ds/2/160/hc49slf-16141.pdf" H 1750 2750 50  0001 C CNN
 F 4 "Mouser" H 1750 2750 60  0001 C CNN "SPR"
-F 5 "559-FOXS080-20-LF" H 1750 2750 60  0001 C CNN "SPN"
-F 6 "Fox" H 0   0   50  0001 C CNN "MFR"
-F 7 "FOXSLF/080-20" H 0   0   50  0001 C CNN "MPN"
-F 8 "" H 0   0   50  0001 C CNN "SPR"
-F 9 "" H 0   0   50  0001 C CNN "SPURL"
+F 5 "815-ABM3B-8.0-10-1UT " H 1750 2750 60  0001 C CNN "SPN"
+F 6 "Abracon" H 0   0   50  0001 C CNN "MFR"
+F 7 "ABM3B-8.000MHZ-10-1UT" H 0   0   50  0001 C CNN "MPN"
 	1    1750 2750
 	0    -1   -1   0
@@
 $EndComp
 $Comp
-L GND #PWR056
+L GND #PWR054
 U 1 1 580219D9
 P 1300 2950
-F 0 "#PWR056" H 1300 2700 50  0001 C CNN
+F 0 "#PWR054" H 1300 2700 50  0001 C CNN
 F 1 "GND" H 1300 2800 50  0000 C CNN
 F 2 "" H 1300 2950 50  0000 C CNN
@@
 $EndComp
 $Comp
-L GND #PWR057
+L GND #PWR055
 U 1 1 580219F7
 P 1300 2550
-F 0 "#PWR057" H 1300 2300 50  0001 C CNN
+F 0 "#PWR055" H 1300 2300 50  0001 C CNN
 F 1 "GND" H 1300 2400 50  0000 C CNN
 F 2 "" H 1300 2550 50  0000 C CNN
@@
 $EndComp
 $Comp
-L GND #PWR058
+L GND #PWR056
 U 1 1 5802210E
 P 1700 1950
-F 0 "#PWR058" H 1700 1700 50  0001 C CNN
+F 0 "#PWR056" H 1700 1700 50  0001 C CNN
 F 1 "GND" H 1700 1800 50  0000 C CNN
 F 2 "" H 1700 1950 50  0000 C CNN
@@
 F 0 "L1" V 6800 1450 50  0000 C CNN
 F 1 "10uH" V 6950 1450 50  0000 C CNN
-F 2 "Resistors_SMD:R_0603" H 6850 1450 50  0001 C CNN
+F 2 "MF_Passives:MF_Passives-L1210" H 6850 1450 50  0001 C CNN
 F 3 "" H 6850 1450 50  0001 C CNN
-F 4 "TDK" H 0   0   50  0001 C CNN "MFR"
+F 4 "Taiyo Yuden" H 0   0   50  0001 C CNN "MFR"
 F 5 "MLZ1608N100L" H 0   0   50  0001 C CNN "MPN"
-F 6 "Mouser" H 0   0   50  0001 C CNN "SPR"
-F 7 "810-MLZ1608N100L" H 0   0   50  0001 C CNN "SPN"
-F 8 "" H 0   0   50  0001 C CNN "SPURL"
+F 6 "Macrofab" H 0   0   50  0001 C CNN "SPR"
+F 7 "MF-IND-1210-10uH" H 0   0   50  0001 C CNN "SPN"
 	1    6850 1450
 	0    -1   -1   0
 $EndComp
 $Comp
-L GND #PWR059
+L GND #PWR057
 U 1 1 58022FD3
 P 8600 1850
-F 0 "#PWR059" H 8600 1600 50  0001 C CNN
+F 0 "#PWR057" H 8600 1600 50  0001 C CNN
 F 1 "GND" H 8600 1700 50  0000 C CNN
 F 2 "" H 8600 1850 50  0000 C CNN
@@
 $EndComp
 $Comp
-L VDD #PWR060
+L VDD #PWR058
 U 1 1 58025E39
 P 3900 900
-F 0 "#PWR060" H 3900 750 50  0001 C CNN
+F 0 "#PWR058" H 3900 750 50  0001 C CNN
 F 1 "VDD" H 3900 1050 50  0000 C CNN
 F 2 "" H 3900 900 50  0000 C CNN
@@
 $EndComp
 $Comp
-L GND #PWR061
+L GND #PWR059
 U 1 1 58026CAB
 P 4000 7000
-F 0 "#PWR061" H 4000 6750 50  0001 C CNN
+F 0 "#PWR059" H 4000 6750 50  0001 C CNN
 F 1 "GND" H 4000 6850 50  0000 C CNN
 F 2 "" H 4000 7000 50  0000 C CNN
@@
 $EndComp
 $Comp
-L VDD #PWR062
+L VDD #PWR060
 U 1 1 58028203
 P 2250 1400
-F 0 "#PWR062" H 2250 1250 50  0001 C CNN
+F 0 "#PWR060" H 2250 1250 50  0001 C CNN
 F 1 "VDD" H 2250 1550 50  0000 C CNN
 F 2 "" H 2250 1400 50  0000 C CNN
@@
 $EndComp
 $Comp
-L GND #PWR063
+L GND #PWR061
 U 1 1 580282E9
 P 2250 1650
-F 0 "#PWR063" H 2250 1400 50  0001 C CNN
+F 0 "#PWR061" H 2250 1400 50  0001 C CNN
 F 1 "GND" H 2250 1500 50  0000 C CNN
 F 2 "" H 2250 1650 50  0000 C CNN
@@
 $EndComp
 $Comp
-L PWR_FLAG #FLG064
+L PWR_FLAG #FLG062
 U 1 1 583894F1
 P 8700 2150
-F 0 "#FLG064" H 8700 2245 50  0001 C CNN
+F 0 "#FLG062" H 8700 2245 50  0001 C CNN
 F 1 "PWR_FLAG" H 8700 2330 50  0000 C CNN
 F 2 "" H 8700 2150 50  0000 C CNN
@@
 $EndComp
 $Comp
-L PWR_FLAG #FLG065
+L PWR_FLAG #FLG063
 U 1 1 5838A45C
 P 8700 1400
-F 0 "#FLG065" H 8700 1495 50  0001 C CNN
+F 0 "#FLG063" H 8700 1495 50  0001 C CNN
 F 1 "PWR_FLAG" H 8700 1580 50  0000 C CNN
 F 2 "" H 8700 1400 50  0000 C CNN
@@
 $EndComp
 $Comp
-L VDD #PWR066
+L VDD #PWR064
 U 1 1 5838BC80
 P 7750 3700
-F 0 "#PWR066" H 7750 3550 50  0001 C CNN
+F 0 "#PWR064" H 7750 3550 50  0001 C CNN
 F 1 "VDD" H 7750 3850 50  0000 C CNN
 F 2 "" H 7750 3700 50  0000 C CNN
@@
 $EndComp
 $Comp
-L VDD #PWR067
+L VDD #PWR065
 U 1 1 5838C666
 P 2250 1100
-F 0 "#PWR067" H 2250 950 50  0001 C CNN
+F 0 "#PWR065" H 2250 950 50  0001 C CNN
 F 1 "VDD" H 2250 1250 50  0000 C CNN
 F 2 "" H 2250 1100 50  0000 C CNN
@@
 $EndComp
 $Comp
-L PWR_FLAG #FLG068
+L PWR_FLAG #FLG066
 U 1 1 5838D3F3
 P 6050 1200
-F 0 "#FLG068" H 6050 1295 50  0001 C CNN
+F 0 "#FLG066" H 6050 1295 50  0001 C CNN
 F 1 "PWR_FLAG" H 6050 1380 50  0000 C CNN
 F 2 "" H 6050 1200 50  0000 C CNN
@@
 $EndComp
 $Comp
-L PWR_FLAG #FLG069
+L PWR_FLAG #FLG067
 U 1 1 5838D677
 P 2550 2300
-F 0 "#FLG069" H 2550 2395 50  0001 C CNN
+F 0 "#FLG067" H 2550 2395 50  0001 C CNN
 F 1 "PWR_FLAG" H 2550 2480 50  0000 C CNN
 F 2 "" H 2550 2300 50  0000 C CNN
@@
 $EndComp
 $Comp
-L PWR_FLAG #FLG070
+L PWR_FLAG #FLG068
 U 1 1 5838D7E4
 P 2850 2200
-F 0 "#FLG070" H 2850 2295 50  0001 C CNN
+F 0 "#FLG068" H 2850 2295 50  0001 C CNN
 F 1 "PWR_FLAG" H 2850 2380 50  0000 C CNN
 F 2 "" H 2850 2200 50  0000 C CNN
@@
 $EndComp
 $Comp
-L GND #PWR071
+L GND #PWR069
 U 1 1 584C78AB
 P 6400 3050
-F 0 "#PWR071" H 6400 2800 50  0001 C CNN
+F 0 "#PWR069" H 6400 2800 50  0001 C CNN
 F 1 "GND" H 6400 2900 50  0000 C CNN
 F 2 "" H 6400 3050 50  0000 C CNN
@@
 $EndComp
 $Comp
-L VDD #PWR072
+L VDD #PWR070
 U 1 1 584C834E
 P 2850 1800
-F 0 "#PWR072" H 2850 1650 50  0001 C CNN
+F 0 "#PWR070" H 2850 1650 50  0001 C CNN
 F 1 "VDD" H 2850 1950 50  0000 C CNN
 F 2 "" H 2850 1800 50  0000 C CNN
@@
 $EndComp
 $Comp
-L VDD #PWR073
+L VDD #PWR071
 U 1 1 584C8473
 P 6400 1100
-F 0 "#PWR073" H 6400 950 50  0001 C CNN
+F 0 "#PWR071" H 6400 950 50  0001 C CNN
 F 1 "VDD" H 6400 1250 50  0000 C CNN
 F 2 "" H 6400 1100 50  0000 C CNN
@@
 $EndComp
 $Comp
-L +3V3 #PWR074
+L +3V3 #PWR072
 U 1 1 584C8AF1
 P 7450 3700
-F 0 "#PWR074" H 7450 3550 50  0001 C CNN
+F 0 "#PWR072" H 7450 3550 50  0001 C CNN
 F 1 "+3V3" H 7450 3840 50  0000 C CNN
 F 2 "" H 7450 3700 50  0000 C CNN

Commit message: new layout
Parts:
- R26, R27, R28, R29, R30, R39, R4: footprint Resistors_SMD:R_0603_HandSoldering -> Resistors_SMD:R_0603
Changed lines of the file:
@@
 F 0 "R27" V 2230 2550 50  0000 C CNN
 F 1 "0" V 2150 2550 50  0000 C CNN
-F 2 "Resistors_SMD:R_0603_HandSoldering" V 2080 2550 50  0001 C CNN
+F 2 "Resistors_SMD:R_0603" V 2080 2550 50  0001 C CNN
 F 3 "" H 2150 2550 50  0001 C CNN
 F 4 "YAGEO" H 0   0   50  0001 C CNN "MFR"
@@
 F 0 "R28" V 2230 2950 50  0000 C CNN
 F 1 "220" V 2150 2950 50  0000 C CNN
-F 2 "Resistors_SMD:R_0603_HandSoldering" V 2080 2950 50  0001 C CNN
+F 2 "Resistors_SMD:R_0603" V 2080 2950 50  0001 C CNN
 F 3 "" H 2150 2950 50  0001 C CNN
 F 4 "YAGEO" H 0   0   50  0001 C CNN "MFR"
@@
 F 0 "R30" V 7580 1450 50  0000 C CNN
 F 1 "47" V 7500 1450 50  0000 C CNN
-F 2 "Resistors_SMD:R_0603_HandSoldering" V 7430 1450 50  0001 C CNN
+F 2 "Resistors_SMD:R_0603" V 7430 1450 50  0001 C CNN
 F 3 "" H 7500 1450 50  0001 C CNN
 F 4 "YAGEO" H 0   0   50  0001 C CNN "MFR"
@@
 F 0 "R29" V 2580 1650 50  0000 C CNN
 F 1 "510" V 2500 1650 50  0000 C CNN
-F 2 "Resistors_SMD:R_0603_HandSoldering" V 2430 1650 50  0001 C CNN
+F 2 "Resistors_SMD:R_0603" V 2430 1650 50  0001 C CNN
 F 3 "" H 2500 1650 50  0001 C CNN
 F 4 "YAGEO" H 0   0   50  0001 C CNN "MFR"
@@
 F 0 "R26" V 2580 1400 50  0000 C CNN
 F 1 "NA" V 2500 1400 50  0000 C CNN
-F 2 "Resistors_SMD:R_0603_HandSoldering" V 2430 1400 50  0001 C CNN
+F 2 "Resistors_SMD:R_0603" V 2430 1400 50  0001 C CNN
 F 3 "" H 2500 1400 50  0001 C CNN
 F 4 "" H 0   0   50  0001 C CNN "MFR"
@@
 F 0 "R4" V 2580 1100 50  0000 C CNN
 F 1 "100k" V 2500 1100 50  0000 C CNN
-F 2 "Resistors_SMD:R_0603_HandSoldering" V 2430 1100 50  0001 C CNN
+F 2 "Resistors_SMD:R_0603" V 2430 1100 50  0001 C CNN
 F 3 "" H 2500 1100 50  0001 C CNN
 F 4 "YAGEO" H 0   0   50  0001 C CNN "MFR"
@@
 F 0 "R39" V 7680 3700 50  0000 C CNN
 F 1 "0" V 7600 3700 50  0000 C CNN
-F 2 "Resistors_SMD:R_0603_HandSoldering" V 7530 3700 50  0001 C CNN
+F 2 "Resistors_SMD:R_0603" V 7530 3700 50  0001 C CNN
 F 3 "" H 7600 3700 50  0001 C CNN
 F 4 "YAGEO" H 0   0   50  0001 C CNN "MFR"

Commit message: Finished new layout
Parts:
- removed C53, C55: 100nF, Capacitors_SMD:C_0402, symbol C
- C19, C20: MFR Murata Electronics -> Yageo; MPN GJM1555C1H200JB1D -> CC0402JRNPO9BN200; SPN 81-GJM1555C1H200JB1D -> 603-CC402JRNPO9BN200
- C54: MFR (none) -> AVX; MPN (none) -> TAJA105K016RNJ; SPN (none) -> 581-TAJA105K016; SPR (none) -> Mouser
Other:
- moved on the sheet: C54

Commit message: Remove 3. LDO some improvements
Parts:
- removed R27: 0, Resistors_SMD:R_0603, symbol R
- added C53: 100nF, Capacitors_SMD:C_0402, symbol C
- added SW1: SW_Push, Buttons_Switches_SMD:SW_SPST_PTS645, symbol SW_Push
- added W39: MCO1, Measurement_Points:Measurement_Point_Round-SMD-Pad_Small, symbol TEST_1P
- C19, C20: value 20pF -> 15pF
- R4: value 100k -> 10k; MPN RC0603JR-07100KL -> RC0603JR-0710KL; SPN 603-RC0603JR-07100KL -> 603-RC0603JR-0710KL
Connections:
- net GND: now also C53.2, SW1.2
- net PA8: now also W39.1
- net at U2.12 (PH0): now also C19.1, Y2.2
- net NRST: now reaches R4.1, U2.14 (NRST)
- net NRST: now also C53.1, SW1.1
Other:
- note added: "MCO1 Testpin"
- note added: "Reset Button"
- moved on the sheet: R4

Commit message: Version 1.2
Parts:
- C19, C20: MFR Yageo -> Vishay; MPN CC0402JRNPO9BN200 -> VJ0402A150FXQCW1BC; SPN 603-CC402JRNPO9BN200 -> 77-VJ0402A150FXQCBC
- L1: value 10uH -> FCM1608KF-601T03; MPN MLZ1608N100L -> BK1608HS601-T; Mouser (none) -> Macrofab; SPN MF-IND-1210-10uH -> 963-BK1608HS601-T; SPR Macrofab -> (none)
- R4: MFR YAGEO -> (none); MPN RC0603JR-0710KL -> (none); SPN 603-RC0603JR-0710KL -> (none); SPR Mouser -> (none)
- SW1: MFR (none) -> C&K Components; MPN (none) -> PTS645SL50SMTR 92 LFS; SPN (none) -> 611-PTS645SL50SMTR92; SPR (none) -> Mouser
Changed lines of the file:
@@
 F 3 "" H 1450 2550 50  0001 C CNN
 F 4 "Mouser" H 1450 2550 60  0001 C CNN "SPR"
-F 5 "603-CC402JRNPO9BN200" H 1450 2550 60  0001 C CNN "SPN"
-F 6 "Yageo" H 0   0   50  0001 C CNN "MFR"
-F 7 "CC0402JRNPO9BN200" H 0   0   50  0001 C CNN "MPN"
-F 8 "" H 0   0   50  0001 C CNN "SPR"
-F 9 "" H 0   0   50  0001 C CNN "SPURL"
+F 5 "77-VJ0402A150FXQCBC" H 1450 2550 60  0001 C CNN "SPN"
+F 6 "Vishay" H 0   0   50  0001 C CNN "MFR"
+F 7 "VJ0402A150FXQCW1BC" H 0   0   50  0001 C CNN "MPN"
+F 8 "" H 0   0   50  0001 C CNN "SPURL"
 	1    1450 2550
 	0    1    1    0
@@
 F 2 "Capacitors_SMD:C_0402" H 1488 2800 50  0001 C CNN
 F 3 "" H 1450 2950 50  0001 C CNN
-F 4 "Yageo" H 0   0   50  0001 C CNN "MFR"
-F 5 "CC0402JRNPO9BN200" H 0   0   50  0001 C CNN "MPN"
-F 6 "Mouser" H 0   0   50  0001 C CNN "SPR"
-F 7 "603-CC402JRNPO9BN200" H 0   0   50  0001 C CNN "SPN"
+F 4 "Vishay" H 0   0   50  0001 C CNN "MFR"
+F 5 "VJ0402A150FXQCW1BC" H 0   0   50  0001 C CNN "MPN"
+F 6 "Mouser" H 0   0   50  0001 C CNN "SPR"
+F 7 "77-VJ0402A150FXQCBC" H 0   0   50  0001 C CNN "SPN"
 F 8 "" H 0   0   50  0001 C CNN "SPURL"
 	1    1450 2950
@@
 P 6850 1450
 F 0 "L1" V 6800 1450 50  0000 C CNN
-F 1 "10uH" V 6950 1450 50  0000 C CNN
+F 1 "FCM1608KF-601T03" V 6950 1450 50  0000 C CNN
 F 2 "MF_Passives:MF_Passives-L1210" H 6850 1450 50  0001 C CNN
 F 3 "" H 6850 1450 50  0001 C CNN
 F 4 "Taiyo Yuden" H 0   0   50  0001 C CNN "MFR"
-F 5 "MLZ1608N100L" H 0   0   50  0001 C CNN "MPN"
-F 6 "Macrofab" H 0   0   50  0001 C CNN "SPR"
-F 7 "MF-IND-1210-10uH" H 0   0   50  0001 C CNN "SPN"
-F 8 "" H 0   0   50  0001 C CNN "SPURL"
+F 5 "BK1608HS601-T" H 0   0   50  0001 C CNN "MPN"
+F 6 "Macrofab" H 0   0   50  0001 C CNN "Mouser"
+F 7 "963-BK1608HS601-T" H 0   0   50  0001 C CNN "SPN"
+F 8 "" H 0   0   50  0001 C CNN "SPR"
+F 9 "" H 0   0   50  0001 C CNN "SPURL"
 	1    6850 1450
 	0    -1   -1   0
@@
 F 2 "Resistors_SMD:R_0603" V 9380 3350 50  0001 C CNN
 F 3 "" H 9450 3350 50  0001 C CNN
-F 4 "YAGEO" H 6950 2250 50  0001 C CNN "MFR"
-F 5 "RC0603JR-0710KL" H 6950 2250 50  0001 C CNN "MPN"
-F 6 "Mouser" H 6950 2250 50  0001 C CNN "SPR"
-F 7 "603-RC0603JR-0710KL" H 6950 2250 50  0001 C CNN "SPN"
+F 4 "" H 6950 2250 50  0001 C CNN "MFR"
+F 5 "" H 6950 2250 50  0001 C CNN "MPN"
+F 6 "" H 6950 2250 50  0001 C CNN "SPR"
+F 7 "" H 6950 2250 50  0001 C CNN "SPN"
+F 8 "" H 0   0   50  0001 C CNN "SPURL"
 	1    9450 3350
 	-1   0    0    1
@@
 F 8 "" H -600 0   50  0001 C CNN "SPURL"
 	1    8650 2600
+	1    0    0    -1
+$EndComp
+$Comp
+L TEST_1P W39
+U 1 1 59E0A8A1
+P 7100 4400
+F 0 "W39" H 7100 4670 50  0000 C CNN
+F 1 "MCO1" H 7100 4600 50  0000 C CNN
+F 2 "Measurement_Points:Measurement_Point_Round-SMD-Pad_Small" H 7300 4400 50  0001 C CNN
+F 3 "" H 7300 4400 50  0000 C CNN
+F 4 "" H 750 500 50  0001 C CNN "MFR"
+F 5 "" H 750 500 50  0001 C CNN "MPN"
+F 6 "" H 750 500 50  0001 C CNN "SPR"
+F 7 "" H 750 500 50  0001 C CNN "SPN"
+F 8 "" H 750 500 50  0001 C CNN "SPURL"
+	1    7100 4400
+	1    0    0    -1
+$EndComp
+$Comp
+L SW_Push SW1
+U 1 1 59E2C3B7
+P 9450 3900
+F 0 "SW1" H 9500 4000 50  0000 L CNN
+F 1 "SW_Push" H 9450 3840 50  0000 C CNN
+F 2 "Buttons_Switches_SMD:SW_SPST_PTS645" H 9450 4100 50  0001 C CNN
+F 3 "" H 9450 4100 50  0001 C CNN
+F 4 "C&K Components" H 0   0   50  0001 C CNN "MFR"
+F 5 "PTS645SL50SMTR 92 LFS" H 0   0   50  0001 C CNN "MPN"
+F 6 "Mouser" H 0   0   50  0001 C CNN "SPR"
+F 7 "611-PTS645SL50SMTR92" H 0   0   50  0001 C CNN "SPN"
+F 8 "" H 0   0   50  0001 C CNN "SPURL"
+	1    9450 3900
+	0    1    1    0
+$EndComp
+$Comp
+L C C53
+U 1 1 59E2C467
+P 9000 3950
+F 0 "C53" H 9025 4050 50  0000 L CNN
+F 1 "100nF" H 9025 3850 50  0000 L CNN
+F 2 "Capacitors_SMD:C_0402" H 9038 3800 50  0001 C CNN
+F 3 "" H 9000 3950 50  0001 C CNN
+F 4 "KEMET" H 700 1350 50  0001 C CNN "MFR"
+F 5 "C0402C104M4RACAUTO" H 700 1350 50  0001 C CNN "MPN"
+F 6 "Mouser" H 700 1350 50  0001 C CNN "SPR"
+F 7 "80-C0402C104M4RAUTO" H 700 1350 50  0001 C CNN "SPN"
+F 8 "" H 700 1350 50  0001 C CNN "SPURL"
+	1    9000 3950
+	1    0    0    -1
+$EndComp
+$Comp
+L VDD #PWR078
+U 1 1 59E2C6BF
+P 9450 3150
+F 0 "#PWR078" H 9450 3000 50  0001 C CNN
+F 1 "VDD" H 9450 3300 50  0000 C CNN
+F 2 "" H 9450 3150 50  0000 C CNN
+F 3 "" H 9450 3150 50  0000 C CNN
+	1    9450 3150
+	1    0    0    -1
+$EndComp
+$Comp
+L GND #PWR079
+U 1 1 59E2C89F
+P 9450 4400
+F 0 "#PWR079" H 9450 4150 50  0001 C CNN
+F 1 "GND" H 9450 4250 50  0000 C CNN
+F 2 "" H 9450 4400 50  0000 C CNN
+F 3 "" H 9450 4400 50  0000 C CNN
+	1    9450 4400
 	1    0    0    -1
 $EndComp
@@
 Text HLabel 5400 6400 2    60   BiDi ~ 0
 PC15
+Text HLabel 7400 4400 2    60   BiDi ~ 0
+PA8
+Text Notes 7000 4550 0    60   ~ 0
+MCO1 Testpin
+Text Label 2500 1100 2    60   ~ 0
+NRST
+Text Label 8600 3600 2    60   ~ 0
+NRST
+Text Notes 8650 4500 0    60   ~ 0
+Reset Button
 Wire Wire Line
 	1750 2600 1750 2550
@@
 Wire Wire Line
 	8650 2900 8650 2750
+Wire Wire Line
+	7400 4400 7100 4400
+Wire Wire Line
+	9000 3800 9000 3600
+Wire Wire Line
+	8600 3600 9450 3600
+Wire Wire Line
+	9450 3500 9450 3700
+Wire Wire Line
+	9000 4100 9000 4250
+Wire Wire Line
+	9000 4250 9450 4250
+Wire Wire Line
+	9450 4100 9450 4400
+Wire Wire Line
+	9450 3150 9450 3200
 Connection ~ 1750 2550
 Connection ~ 1750 2950
@@
 Connection ~ 8300 2350
 Connection ~ 8300 2900
-Text HLabel 7400 4400 2    60   BiDi ~ 0
-PA8
-$Comp
-L TEST_1P W39
-U 1 1 59E0A8A1
-P 7100 4400
-F 0 "W39" H 7100 4670 50  0000 C CNN
-F 1 "MCO1" H 7100 4600 50  0000 C CNN
-F 2 "Measurement_Points:Measurement_Point_Round-SMD-Pad_Small" H 7300 4400 50  0001 C CNN
-F 3 "" H 7300 4400 50  0000 C CNN
-F 4 "" H 750 500 50  0001 C CNN "MFR"
-F 5 "" H 750 500 50  0001 C CNN "MPN"
-F 6 "" H 750 500 50  0001 C CNN "SPR"
-F 7 "" H 750 500 50  0001 C CNN "SPN"
-F 8 "" H 750 500 50  0001 C CNN "SPURL"
-	1    7100 4400
-	1    0    0    -1
-$EndComp
-Wire Wire Line
-	7400 4400 7100 4400
-Text Notes 7000 4550 0    60   ~ 0
-MCO1 Testpin
-$Comp
-L SW_Push SW1
-U 1 1 59E2C3B7
-P 9450 3900
-F 0 "SW1" H 9500 4000 50  0000 L CNN
-F 1 "SW_Push" H 9450 3840 50  0000 C CNN
-F 2 "Buttons_Switches_SMD:SW_SPST_PTS645" H 9450 4100 50  0001 C CNN
-F 3 "" H 9450 4100 50  0001 C CNN
-	1    9450 3900
-	0    1    1    0
-$EndComp
-$Comp
-L C C53
-U 1 1 59E2C467
-P 9000 3950
-F 0 "C53" H 9025 4050 50  0000 L CNN
-F 1 "100nF" H 9025 3850 50  0000 L CNN
-F 2 "Capacitors_SMD:C_0402" H 9038 3800 50  0001 C CNN
-F 3 "" H 9000 3950 50  0001 C CNN
-F 4 "KEMET" H 700 1350 50  0001 C CNN "MFR"
-F 5 "C0402C104M4RACAUTO" H 700 1350 50  0001 C CNN "MPN"
-F 6 "Mouser" H 700 1350 50  0001 C CNN "SPR"
-F 7 "80-C0402C104M4RAUTO" H 700 1350 50  0001 C CNN "SPN"
-F 8 "" H 700 1350 50  0001 C CNN "SPURL"
-	1    9000 3950
-	1    0    0    -1
-$EndComp
-$Comp
-L VDD #PWR078
-U 1 1 59E2C6BF
-P 9450 3150
-F 0 "#PWR078" H 9450 3000 50  0001 C CNN
-F 1 "VDD" H 9450 3300 50  0000 C CNN
-F 2 "" H 9450 3150 50  0000 C CNN
-F 3 "" H 9450 3150 50  0000 C CNN
-	1    9450 3150
-	1    0    0    -1
-$EndComp
-Wire Wire Line
-	9000 3800 9000 3600
-Wire Wire Line
-	8600 3600 9450 3600
-Wire Wire Line
-	9450 3500 9450 3700
 Connection ~ 9450 3600
-Wire Wire Line
-	9000 4100 9000 4250
-Wire Wire Line
-	9000 4250 9450 4250
-Wire Wire Line
-	9450 4100 9450 4400
-$Comp
-L GND #PWR079
-U 1 1 59E2C89F
-P 9450 4400
-F 0 "#PWR079" H 9450 4150 50  0001 C CNN
-F 1 "GND" H 9450 4250 50  0000 C CNN
-F 2 "" H 9450 4400 50  0000 C CNN
-F 3 "" H 9450 4400 50  0000 C CNN
-	1    9450 4400
-	1    0    0    -1
-$EndComp
 Connection ~ 9450 4250
-Text Label 2500 1100 2    60   ~ 0
-NRST
-Text Label 8600 3600 2    60   ~ 0
-NRST
 Connection ~ 9000 3600
-Wire Wire Line
-	9450 3150 9450 3200
-Text Notes 8650 4500 0    60   ~ 0
-Reset Button
 $EndSCHEMATC
