File: Main.sch (KiCad schematic (older format))
At the start: 27 parts, among them SW1 SW_Push, U2 STM32F407VGTx, Y2 8MHz

Commit message: Fixed footprint of L1
Parts:
- L1: footprint MF_Passives:MF_Passives-L1210 -> Resistors_SMD:R_0603
Changed lines of the file:
@@
 F 0 "L1" V 6800 1450 50  0000 C CNN
 F 1 "FCM1608KF-601T03" V 6950 1450 50  0000 C CNN
-F 2 "MF_Passives:MF_Passives-L1210" H 6850 1450 50  0001 C CNN
+F 2 "Resistors_SMD:R_0603" H 6850 1450 50  0001 C CNN
 F 3 "" H 6850 1450 50  0001 C CNN
 F 4 "Taiyo Yuden" H 0   0   50  0001 C CNN "MFR"
@@
 F 6 "Macrofab" H 0   0   50  0001 C CNN "Mouser"
 F 7 "963-BK1608HS601-T" H 0   0   50  0001 C CNN "SPN"
-F 8 "" H 0   0   50  0001 C CNN "SPR"
-F 9 "" H 0   0   50  0001 C CNN "SPURL"
 	1    6850 1450
 	0    -1   -1   0
