File: VS1053.sch (KiCad schematic (older format))
At the start: 44 parts, among them U1 VS1053, U7 STEREO-AUDIO-JACK, Y1 12.288 Mhz

Commit message: VS1053: use kicad audio jack component
Parts:
- removed U7: STEREO-AUDIO-JACK, jfi:AUDIO_JACK, symbol STEREO-AUDIO-JACK
- added U7: LINEOUT, symbol Audio-Jack-3_2Switches
Connections:
- wire segments 116 -> 165
Other:
- moved on the sheet: C17, C18, C24, C25, C26, C27, R40, R41, R42, R43, R6, R7

Commit message: Use smd oscilator Add testpoints Use different power networks
Parts:
- added W10, W6: SCLK, Measurement_Points:Measurement_Point_Round-SMD-Pad_Small, symbol TEST_1P
- added W11: MCLK, Measurement_Points:Measurement_Point_Round-SMD-Pad_Small, symbol TEST_1P
- added W12: XRESET, Measurement_Points:Measurement_Point_Round-SMD-Pad_Small, symbol TEST_1P
- added W13: LROUT, Measurement_Points:Measurement_Point_Round-SMD-Pad_Small, symbol TEST_1P
- added W4: MISO, Measurement_Points:Measurement_Point_Round-SMD-Pad_Small, symbol TEST_1P
- added W5: MOSI, Measurement_Points:Measurement_Point_Round-SMD-Pad_Small, symbol TEST_1P
- added W7: XCS, Measurement_Points:Measurement_Point_Round-SMD-Pad_Small, symbol TEST_1P
- added W8: SDATA, Measurement_Points:Measurement_Point_Round-SMD-Pad_Small, symbol TEST_1P
- added W9: XDCS, Measurement_Points:Measurement_Point_Round-SMD-Pad_Small, symbol TEST_1P
- C1, C2, C24, C25: footprint Capacitors_SMD:C_0603_HandSoldering -> Capacitors_SMD:C_0603
- C26, C27: value 10uF -> 75uF
- Y1: footprint Crystals:Crystal_HC49-U_Vertical -> Crystals:Crystal_SMD_ABM3B; MPN ABL-12.288MHZ-B2 -> ABM3B-12.288MHZ-10-1-U-T; SPN 815-ABL-12.288-B2 -> 815-ABM3B-12.288-T
Connections:
- net labels added: +3.3VA, LEFT, RIGHT
- wire segments 165 -> 125
Other:
- moved on the sheet: C1, C16, C17, C18, C2, C24, C25, C26, C27, R1, R33, R35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

Commit message: new layout
Parts:
- removed JP1, JP2: JUMPER, Capacitors_SMD:C_0603, symbol JUMPER
- R1, R2, R3, R40, R41, R42, R43, R5, R6, R7: footprint Resistors_SMD:R_0603_HandSoldering -> Resistors_SMD:R_0603
- U7: footprint (none) -> jfi:AUDIO_JACK
Connections:
- net labels removed: SCL, SDA, VS_SCL, VS_SDA
- wire segments 125 -> 123
Changed lines of the file:
@@
 F 0 "R1" V 3380 5100 50  0000 C CNN
 F 1 "1M" V 3300 5100 50  0000 C CNN
-F 2 "Resistors_SMD:R_0603_HandSoldering" V 3230 5100 50  0001 C CNN
+F 2 "Resistors_SMD:R_0603" V 3230 5100 50  0001 C CNN
 F 3 "" H 3300 5100 50  0001 C CNN
 F 4 "Mouser" V 3300 5100 60  0001 C CNN "SP"
@@
 F 0 "R2" V 3730 4550 50  0000 C CNN
 F 1 "100k" V 3650 4550 50  0000 C CNN
-F 2 "Resistors_SMD:R_0603_HandSoldering" V 3580 4550 50  0001 C CNN
+F 2 "Resistors_SMD:R_0603" V 3580 4550 50  0001 C CNN
 F 3 "" H 3650 4550 50  0001 C CNN
 F 4 "YAGEO" H 0   0   50  0001 C CNN "MFR"
@@
 F 0 "R3" V 3830 6800 50  0000 C CNN
 F 1 "100k" V 3750 6800 50  0000 C CNN
-F 2 "Resistors_SMD:R_0603_HandSoldering" V 3680 6800 50  0001 C CNN
+F 2 "Resistors_SMD:R_0603" V 3680 6800 50  0001 C CNN
 F 3 "" H 3750 6800 50  0001 C CNN
 F 4 "YAGEO" H 0   0   50  0001 C CNN "MFR"
@@
 F 0 "R5" V 6480 5600 50  0000 C CNN
 F 1 "10R" V 6400 5600 50  0000 C CNN
-F 2 "Resistors_SMD:R_0603_HandSoldering" V 6330 5600 50  0001 C CNN
+F 2 "Resistors_SMD:R_0603" V 6330 5600 50  0001 C CNN
 F 3 "" H 6400 5600 50  0001 C CNN
 F 4 "YAGEO" H -2000 0   50  0001 C CNN "MFR"
@@
 F 0 "R6" V 8580 2600 50  0000 C CNN
 F 1 "20R" V 8500 2600 50  0000 C CNN
-F 2 "Resistors_SMD:R_0603_HandSoldering" V 8430 2600 50  0001 C CNN
+F 2 "Resistors_SMD:R_0603" V 8430 2600 50  0001 C CNN
 F 3 "" H 8500 2600 50  0001 C CNN
 F 4 "YAGEO" H 300 0   50  0001 C CNN "MFR"
@@
 F 0 "R7" V 8580 3500 50  0000 C CNN
 F 1 "20R" V 8500 3500 50  0000 C CNN
-F 2 "Resistors_SMD:R_0603_HandSoldering" V 8430 3500 50  0001 C CNN
+F 2 "Resistors_SMD:R_0603" V 8430 3500 50  0001 C CNN
 F 3 "" H 8500 3500 50  0001 C CNN
 F 4 "YAGEO" H 300 600 50  0001 C CNN "MFR"
@@
 $EndComp
 $Comp
-L JUMPER JP1
-U 1 1 5802FA80
-P 1900 7200
-F 0 "JP1" H 1900 7350 50  0000 C CNN
-F 1 "JUMPER" H 1900 7120 50  0000 C CNN
-F 2 "Capacitors_SMD:C_0603" H 1900 7200 50  0001 C CNN
-F 3 "" H 1900 7200 50  0000 C CNN
-F 4 "" H -50 300 50  0001 C CNN "MFR"
-F 5 "" H -50 300 50  0001 C CNN "MPN"
-F 6 "" H -50 300 50  0001 C CNN "SPR"
-F 7 "" H -50 300 50  0001 C CNN "SPN"
-F 8 "" H -50 300 50  0001 C CNN "SPURL"
-	1    1900 7200
-	1    0    0    -1
-$EndComp
-$Comp
-L JUMPER JP2
-U 1 1 5802FB4F
-P 1900 7550
-F 0 "JP2" H 1900 7700 50  0000 C CNN
-F 1 "JUMPER" H 1900 7470 50  0000 C CNN
-F 2 "Capacitors_SMD:C_0603" H 1900 7550 50  0001 C CNN
-F 3 "" H 1900 7550 50  0000 C CNN
-F 4 "" H -50 300 50  0001 C CNN "MFR"
-F 5 "" H -50 300 50  0001 C CNN "MPN"
-F 6 "" H -50 300 50  0001 C CNN "SPR"
-F 7 "" H -50 300 50  0001 C CNN "SPN"
-F 8 "" H -50 300 50  0001 C CNN "SPURL"
-	1    1900 7550
-	1    0    0    -1
-$EndComp
-$Comp
 L GND #PWR07
 U 1 1 58353245
@@
 F 0 "R40" V 8980 3250 50  0000 C CNN
 F 1 "470" V 8900 3250 50  0000 C CNN
-F 2 "Resistors_SMD:R_0603_HandSoldering" V 8830 3250 50  0001 C CNN
+F 2 "Resistors_SMD:R_0603" V 8830 3250 50  0001 C CNN
 F 3 "" H 8900 3250 50  0001 C CNN
 F 4 "YAGEO" H 1000 2450 50  0001 C CNN "MFR"
@@
 F 0 "R42" V 9880 3500 50  0000 C CNN
 F 1 "100k" V 9800 3500 50  0000 C CNN
-F 2 "Resistors_SMD:R_0603_HandSoldering" V 9730 3500 50  0001 C CNN
+F 2 "Resistors_SMD:R_0603" V 9730 3500 50  0001 C CNN
 F 3 "" H 9800 3500 50  0001 C CNN
 F 4 "YAGEO" H 1000 2450 50  0001 C CNN "MFR"
@@
 F 0 "R41" V 8980 2850 50  0000 C CNN
 F 1 "470" V 8900 2850 50  0000 C CNN
-F 2 "Resistors_SMD:R_0603_HandSoldering" V 8830 2850 50  0001 C CNN
+F 2 "Resistors_SMD:R_0603" V 8830 2850 50  0001 C CNN
 F 3 "" H 8900 2850 50  0001 C CNN
 F 4 "YAGEO" H 1000 1250 50  0001 C CNN "MFR"
@@
 F 0 "R43" V 9880 2450 50  0000 C CNN
 F 1 "100k" V 9800 2450 50  0000 C CNN
-F 2 "Resistors_SMD:R_0603_HandSoldering" V 9730 2450 50  0001 C CNN
+F 2 "Resistors_SMD:R_0603" V 9730 2450 50  0001 C CNN
 F 3 "" H 9800 2450 50  0001 C CNN
 F 4 "YAGEO" H 1000 600 50  0001 C CNN "MFR"
@@
 Text HLabel 6750 4100 2    60   Output ~ 0
 VS_UART_TX
-Text HLabel 1600 7550 0    60   Input ~ 0
-VS_SDA
-Text HLabel 1600 7200 0    60   Input ~ 0
-VS_SCL
-Text Label 3350 6050 2    60   ~ 0
-SCL
-Text Label 3350 6150 2    60   ~ 0
-SDA
-Text Label 2550 7200 0    60   ~ 0
-SCL
-Text Label 2500 7550 0    60   ~ 0
-SDA
 Text Label 6500 850  0    60   ~ 0
 CVDD
@@
 Wire Wire Line
 	1950 6550 3900 6550
-Wire Wire Line
-	3900 6050 3350 6050
-Wire Wire Line
-	3350 6150 3900 6150
-Wire Wire Line
-	2550 7200 2200 7200
-Wire Wire Line
-	2200 7550 2500 7550
 Wire Wire Line
 	5800 4100 6750 4100
@@
 F 0 "U7" H 10500 3290 50  0000 C CNN
 F 1 "LINEOUT" H 10350 2800 50  0000 L CNN
-F 2 "" H 10750 3100 50  0001 C CNN
+F 2 "jfi:AUDIO_JACK" H 10750 3100 50  0001 C CNN
 F 3 "" H 10750 3100 50  0001 C CNN
 	1    10500 3000
@@
 	4800 1150 6300 1150
 Connection ~ 5300 1150
+Wire Wire Line
+	3900 6050 3750 6050
+Connection ~ 3750 6050
+Wire Wire Line
+	3900 6150 3750 6150
+Connection ~ 3750 6150
 $EndSCHEMATC

Commit message: Finished new layout
Parts:
- added R56: 100k, Resistors_SMD:R_0603, symbol R
- C15: MFR (none) -> AVX; MPN (none) -> TAJA105K016RNJ; SPN (none) -> 581-TAJA105K016; SPR (none) -> Mouser
- U7: MFR (none) -> CUI; MPN (none) -> SJ1-3535NG; SPN (none) -> 490-SJ1-3535NG; SPR (none) -> Mouser
Connections:
- net GND: now also R56.2
- net at R3.1, U1.33 (GPIO0), U1.34 (GPIO1): no longer U1.10 (GPIO3/SDATA), U1.9 (GPIO2/DCLK)
- new net: R56.1, U1.10 (GPIO3/SDATA), U1.9 (GPIO2/DCLK)
Other:
- moved on the sheet: R3

Commit message: Remove 3. LDO some improvements
Parts:
- added R57: 0, Resistors_SMD:R_0603, symbol R
- C1, C2: value 33pF -> 15pF
- C26, C27: value 75uF -> 10uF
Connections:
- net +3.3VA is gone; now on net +3V3: R34.2
- net GND: now also R57.2; no longer C10.2, C13.2, C15.2, C16.1, C17.2, C18.1, C24.2, C25.2, C4.2, C7.2, R42.1, R43.1, U1.37 (AGND), U1.40 (AGND), U1.41 (AGND), U1.47 (AGND), U7.3
- new net GNDA: C10.2, C13.2, C15.2, C16.1, C17.2, C18.1, C24.2, C25.2, C4.2, C7.2, R42.1, R43.1, R57.1, U1.37 (AGND), U1.40 (AGND), U1.41 (AGND), U1.47 (AGND), U7.3
Other:
- moved on the sheet: R33, R34, R35

Commit message: some minor improvements
Parts:
- added R27, R58, R59, R60: NA, Resistors_SMD:R_0603, symbol R
- added RV1, RV2: POT_TRIM, Potentiometers:Potentiometer_WirePads_Small, symbol POT_TRIM
Connections:
- net GNDA: now also R59.1, R60.2, RV1.3, RV2.1
- net at C26.2, R42.2: now also R58.1, RV2.3; no longer U7.2
- net at C27.2, R43.2: now also R27.2, RV1.1; no longer U7.1
- new net: R27.1, R59.2, RV1.2, U7.1
- new net: R58.2, R60.1, RV2.2, U7.2
Other:
- moved on the sheet: C17, C18, C24, C25, C26, C27, R40, R41, R42, R43, R6, R7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

Commit message: Version 1.2
Parts:
- C1, C2: footprint Capacitors_SMD:C_0603 -> Capacitors_SMD:C_0402; MFR Murata Electronics -> Vishay; MPN GRM1885C1H330JA01D -> VJ0402A150FXQCW1BC; SP Mouser -> (none); SPN 81-GRM39C330J50 -> 77-VJ0402A150FXQCBC; Vishay (none) -> Murata Electronics
- C26, C27: footprint Capacitors_SMD:c_elec_5x5.7 -> Capacitors_SMD:c_elec_4x5.7
- R27, R58: value NA -> 0
- RV1, RV2: value POT_TRIM -> 10k
