File: VS1053.sch (KiCad schematic (older format))
At the start: 60 parts, among them U1 VS1053, U7 LINEOUT, Y1 12.288 Mhz

Commit message: Changed butten connectors
Parts:
- added R25, R32: 100k, Resistors_SMD:R_0603, symbol R
- RV1, RV2: footprint Potentiometers:Potentiometer_WirePads_Small -> jfi:Potentiometer_WirePads_Small_nosilk
Connections:
- net GND: now also R25.2, R32.2
- net at R56.1, U1.10 (GPIO3/SDATA): no longer U1.9 (GPIO2/DCLK)
- net +3V3 renamed +3.3VA
- new net: R25.1, U1.33 (GPIO0)
- new net: R32.1, U1.34 (GPIO1)
- new net: R3.1, U1.9 (GPIO2/DCLK)
Other:
- moved on the sheet: R3, R56
