File: externals.sch (KiCad schematic (older format))
At the start: 78 parts, among them J1 SWD, J2 RC522_Header, J3 Screw_Terminal_1x02, P2 VolDown, P3 Prev, P4 Play, P5 Next, P6 VolUp, P7 CONN_02X10, Q1 BSS138

Commit message: Version 1.2
Parts:
- C48: value 75uF -> 10uF; footprint Capacitors_SMD:c_elec_5x5.7 -> Capacitors_SMD:c_elec_4x5.7
- R16, R18, R19, R20, R21, R22, R25, R32: MFR YAGEO -> (none); MPN RC0603JR-0710KL -> (none); SPN 603-RC0603JR-0710KL -> (none); SPR Mouser -> (none)
Changed lines of the file:
@@
 F 2 "Resistors_SMD:R_0603" V 8430 3850 50  0001 C CNN
 F 3 "" H 8500 3850 50  0001 C CNN
-F 4 "YAGEO" H 150 850 50  0001 C CNN "MFR"
-F 5 "RC0603JR-0710KL" H 150 850 50  0001 C CNN "MPN"
-F 6 "Mouser" H 150 850 50  0001 C CNN "SPR"
-F 7 "603-RC0603JR-0710KL" H 150 850 50  0001 C CNN "SPN"
+F 4 "" H 150 850 50  0001 C CNN "MFR"
+F 5 "" H 150 850 50  0001 C CNN "MPN"
+F 6 "" H 150 850 50  0001 C CNN "SPR"
+F 7 "" H 150 850 50  0001 C CNN "SPN"
 F 8 "" H 150 850 50  0001 C CNN "SPURL"
 	1    8500 3850
@@
 F 2 "Resistors_SMD:R_0603" V 8630 3850 50  0001 C CNN
 F 3 "" H 8700 3850 50  0001 C CNN
-F 4 "YAGEO" H 150 850 50  0001 C CNN "MFR"
-F 5 "RC0603JR-0710KL" H 150 850 50  0001 C CNN "MPN"
-F 6 "Mouser" H 150 850 50  0001 C CNN "SPR"
-F 7 "603-RC0603JR-0710KL" H 150 850 50  0001 C CNN "SPN"
+F 4 "" H 150 850 50  0001 C CNN "MFR"
+F 5 "" H 150 850 50  0001 C CNN "MPN"
+F 6 "" H 150 850 50  0001 C CNN "SPR"
+F 7 "" H 150 850 50  0001 C CNN "SPN"
 F 8 "" H 150 850 50  0001 C CNN "SPURL"
 	1    8700 3850
@@
 F 2 "Resistors_SMD:R_0603" V 8830 3850 50  0001 C CNN
 F 3 "" H 8900 3850 50  0001 C CNN
-F 4 "YAGEO" H 150 850 50  0001 C CNN "MFR"
-F 5 "RC0603JR-0710KL" H 150 850 50  0001 C CNN "MPN"
-F 6 "Mouser" H 150 850 50  0001 C CNN "SPR"
-F 7 "603-RC0603JR-0710KL" H 150 850 50  0001 C CNN "SPN"
+F 4 "" H 150 850 50  0001 C CNN "MFR"
+F 5 "" H 150 850 50  0001 C CNN "MPN"
+F 6 "" H 150 850 50  0001 C CNN "SPR"
+F 7 "" H 150 850 50  0001 C CNN "SPN"
 F 8 "" H 150 850 50  0001 C CNN "SPURL"
 	1    8900 3850
@@
 F 2 "Resistors_SMD:R_0603" V 8230 3850 50  0001 C CNN
 F 3 "" H 8300 3850 50  0001 C CNN
-F 4 "YAGEO" H 150 850 50  0001 C CNN "MFR"
-F 5 "RC0603JR-0710KL" H 150 850 50  0001 C CNN "MPN"
-F 6 "Mouser" H 150 850 50  0001 C CNN "SPR"
-F 7 "603-RC0603JR-0710KL" H 150 850 50  0001 C CNN "SPN"
+F 4 "" H 150 850 50  0001 C CNN "MFR"
+F 5 "" H 150 850 50  0001 C CNN "MPN"
+F 6 "" H 150 850 50  0001 C CNN "SPR"
+F 7 "" H 150 850 50  0001 C CNN "SPN"
 F 8 "" H 150 850 50  0001 C CNN "SPURL"
 	1    8300 3850
@@
 F 2 "Resistors_SMD:R_0603" V 8030 3850 50  0001 C CNN
 F 3 "" H 8100 3850 50  0001 C CNN
-F 4 "YAGEO" H 150 850 50  0001 C CNN "MFR"
-F 5 "RC0603JR-0710KL" H 150 850 50  0001 C CNN "MPN"
-F 6 "Mouser" H 150 850 50  0001 C CNN "SPR"
-F 7 "603-RC0603JR-0710KL" H 150 850 50  0001 C CNN "SPN"
+F 4 "" H 150 850 50  0001 C CNN "MFR"
+F 5 "" H 150 850 50  0001 C CNN "MPN"
+F 6 "" H 150 850 50  0001 C CNN "SPR"
+F 7 "" H 150 850 50  0001 C CNN "SPN"
 F 8 "" H 150 850 50  0001 C CNN "SPURL"
 	1    8100 3850
@@
 F 2 "Resistors_SMD:R_0603" V 7830 3850 50  0001 C CNN
 F 3 "" H 7900 3850 50  0001 C CNN
-F 4 "YAGEO" H 150 850 50  0001 C CNN "MFR"
-F 5 "RC0603JR-0710KL" H 150 850 50  0001 C CNN "MPN"
-F 6 "Mouser" H 150 850 50  0001 C CNN "SPR"
-F 7 "603-RC0603JR-0710KL" H 150 850 50  0001 C CNN "SPN"
+F 4 "" H 150 850 50  0001 C CNN "MFR"
+F 5 "" H 150 850 50  0001 C CNN "MPN"
+F 6 "" H 150 850 50  0001 C CNN "SPR"
+F 7 "" H 150 850 50  0001 C CNN "SPN"
 F 8 "" H 150 850 50  0001 C CNN "SPURL"
 	1    7900 3850
@@
 F 2 "Resistors_SMD:R_0603" V 2980 1000 50  0001 C CNN
 F 3 "" H 3050 1000 50  0001 C CNN
-F 4 "YAGEO" H 0   0   50  0001 C CNN "MFR"
-F 5 "RC0603JR-0710KL" H 0   0   50  0001 C CNN "MPN"
-F 6 "Mouser" H 0   0   50  0001 C CNN "SPR"
-F 7 "603-RC0603JR-0710KL" H 0   0   50  0001 C CNN "SPN"
+F 4 "" H 0   0   50  0001 C CNN "MFR"
+F 5 "" H 0   0   50  0001 C CNN "MPN"
+F 6 "" H 0   0   50  0001 C CNN "SPR"
+F 7 "" H 0   0   50  0001 C CNN "SPN"
 F 8 "" H 0   0   50  0001 C CNN "SPURL"
 	1    3050 1000
@@
 P 750 1350
 F 0 "C48" H 775 1450 50  0000 L CNN
-F 1 "75uF" H 775 1250 50  0000 L CNN
-F 2 "Capacitors_SMD:c_elec_5x5.7" H 788 1200 50  0001 C CNN
+F 1 "10uF" H 775 1250 50  0000 L CNN
+F 2 "Capacitors_SMD:c_elec_4x5.7" H 788 1200 50  0001 C CNN
 F 3 "" H 750 1350 50  0001 C CNN
 F 4 "Panasonic" H 0   0   50  0001 C CNN "MFR"
@@
 F 6 "Mouser" H 0   0   50  0001 C CNN "SPR"
 F 7 "667-EEE-HD1V100AR" H 0   0   50  0001 C CNN "SPN"
-F 8 "" H 0   0   50  0001 C CNN "SPURL"
 	1    750  1350
 	1    0    0    -1
@@
 F 2 "Resistors_SMD:R_0603" V 3630 1000 50  0001 C CNN
 F 3 "" H 3700 1000 50  0001 C CNN
-F 4 "YAGEO" H 0   0   50  0001 C CNN "MFR"
-F 5 "RC0603JR-0710KL" H 0   0   50  0001 C CNN "MPN"
-F 6 "Mouser" H 0   0   50  0001 C CNN "SPR"
-F 7 "603-RC0603JR-0710KL" H 0   0   50  0001 C CNN "SPN"
+F 4 "" H 0   0   50  0001 C CNN "MFR"
+F 5 "" H 0   0   50  0001 C CNN "MPN"
+F 6 "" H 0   0   50  0001 C CNN "SPR"
+F 7 "" H 0   0   50  0001 C CNN "SPN"
 F 8 "" H 0   0   50  0001 C CNN "SPURL"
 	1    3700 1000
@@
 F 3 "" H 9500 5200 50  0000 C CNN
 	1    9500 5200
+	1    0    0    -1
+$EndComp
+$Comp
+L D_Schottky D8
+U 1 1 59E06461
+P 2100 5950
+F 0 "D8" H 2100 6050 50  0000 C CNN
+F 1 "D_Schottky_30_V_3A" H 2100 5850 50  0000 C CNN
+F 2 "Diodes_SMD:SMB_Standard" H 2100 5950 50  0001 C CNN
+F 3 "" H 2100 5950 50  0001 C CNN
+F 4 "Mouser" H 2100 5950 60  0001 C CNN "SPR"
+F 5 "621-B330-F" H 2100 5950 60  0001 C CNN "SPN"
+F 6 "Diodes Incorporated" H -1250 3150 50  0001 C CNN "MFR"
+F 7 "B330-13-F" H -1250 3150 50  0001 C CNN "MPN"
+F 8 "" H -1250 3150 50  0001 C CNN "SPR"
+F 9 "" H -1250 3150 50  0001 C CNN "SPURL"
+	1    2100 5950
+	1    0    0    -1
+$EndComp
+$Comp
+L Conn_02x04_Counter_Clockwise J1
+U 1 1 59E2A8F8
+P 1600 4600
+F 0 "J1" H 1650 4800 50  0000 C CNN
+F 1 "SWD" H 1650 4300 50  0000 C CNN
+F 2 "Pin_Headers:Pin_Header_Straight_2x04" H 1600 4600 50  0001 C CNN
+F 3 "" H 1600 4600 50  0001 C CNN
+F 4 "" H 0   0   50  0001 C CNN "MFR"
+F 5 "" H 0   0   50  0001 C CNN "MPN"
+F 6 "" H 0   0   50  0001 C CNN "SPR"
+F 7 "" H 0   0   50  0001 C CNN "SPN"
+F 8 "" H 0   0   50  0001 C CNN "SPURL"
+	1    1600 4600
 	1    0    0    -1
 $EndComp
@@
 Text Label 3700 700  2    60   ~ 0
 BTLED_NET_5V
+Text HLabel 2000 4700 2    60   BiDi ~ 0
+DBG_RX
+Text HLabel 2000 4800 2    60   BiDi ~ 0
+DBG_TX
 Wire Wire Line
 	2800 3450 2550 3450
@@
 Wire Wire Line
 	9500 4850 9500 5200
+Wire Wire Line
+	2450 5950 2250 5950
+Wire Wire Line
+	2450 6150 1750 6150
+Wire Wire Line
+	1950 5950 1750 5950
+Wire Wire Line
+	1400 4600 1300 4600
+Wire Wire Line
+	1300 4700 1400 4700
+Wire Wire Line
+	1400 4800 1300 4800
+Wire Wire Line
+	1300 4800 1300 4850
+Wire Wire Line
+	1400 4500 1300 4500
+Wire Wire Line
+	1300 4500 1300 4450
+Wire Wire Line
+	2000 4700 1900 4700
+Wire Wire Line
+	2000 4800 1900 4800
 Connection ~ 2800 3150
 Connection ~ 2800 2850
@@
 Connection ~ 9100 3500
 NoConn ~ 10550 1450
-$Comp
-L D_Schottky D8
-U 1 1 59E06461
-P 2100 5950
-F 0 "D8" H 2100 6050 50  0000 C CNN
-F 1 "D_Schottky_30_V_3A" H 2100 5850 50  0000 C CNN
-F 2 "Diodes_SMD:SMB_Standard" H 2100 5950 50  0001 C CNN
-F 3 "" H 2100 5950 50  0001 C CNN
-F 4 "Mouser" H 2100 5950 60  0001 C CNN "SPR"
-F 5 "621-B330-F" H 2100 5950 60  0001 C CNN "SPN"
-F 6 "Diodes Incorporated" H -1250 3150 50  0001 C CNN "MFR"
-F 7 "B330-13-F" H -1250 3150 50  0001 C CNN "MPN"
-F 8 "" H -1250 3150 50  0001 C CNN "SPR"
-F 9 "" H -1250 3150 50  0001 C CNN "SPURL"
-	1    2100 5950
-	1    0    0    -1
-$EndComp
-Wire Wire Line
-	2450 5950 2250 5950
-Wire Wire Line
-	2450 6150 1750 6150
-Wire Wire Line
-	1950 5950 1750 5950
-$Comp
-L Conn_02x04_Counter_Clockwise J1
-U 1 1 59E2A8F8
-P 1600 4600
-F 0 "J1" H 1650 4800 50  0000 C CNN
-F 1 "SWD" H 1650 4300 50  0000 C CNN
-F 2 "Pin_Headers:Pin_Header_Straight_2x04" H 1600 4600 50  0001 C CNN
-F 3 "" H 1600 4600 50  0001 C CNN
-	1    1600 4600
-	1    0    0    -1
-$EndComp
-Wire Wire Line
-	1400 4600 1300 4600
-Wire Wire Line
-	1300 4700 1400 4700
-Wire Wire Line
-	1400 4800 1300 4800
-Wire Wire Line
-	1300 4800 1300 4850
-Wire Wire Line
-	1400 4500 1300 4500
-Wire Wire Line
-	1300 4500 1300 4450
-Text HLabel 2000 4700 2    60   BiDi ~ 0
-DBG_RX
-Text HLabel 2000 4800 2    60   BiDi ~ 0
-DBG_TX
-Wire Wire Line
-	2000 4700 1900 4700
-Wire Wire Line
-	2000 4800 1900 4800
 NoConn ~ 1900 4500
 NoConn ~ 1900 4600
